File: turrismox-dsdshu-adapter.kicad_sch (KiCad schematic)
At the start: 2 parts, among them J1 Conn_01x06, J2 Conn_02x17_Odd_Even

Commit message: set plotting settings, add mounting hole footprint
Parts:
- J1: LCSC (none) -> C492238
- J2: LCSC (none) -> C2685114
Changed lines of the file:
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@@
+      (effects (font (size 1.27 1.27)) hide)
+    )
+    (property "LCSC" "C2685114" (id 4) (at 123.19 60.96 90)
       (effects (font (size 1.27 1.27)) hide)
     )
@@
       (effects (font (size 1.27 1.27)) hide)
     )
+    (property "LCSC" "C492238" (id 4) (at 175.26 62.23 0)
+      (effects (font (size 1.27 1.27)) hide)
+    )

Commit message: change design to use ribbon cable for Mox connection
Parts:
- J2: footprint footprints:Liansheng FH-00357 -> footprints:Ckmtw_B-3000N34P-0110; LCSC C2685114 -> C383613
Changed lines of the file:
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@@
       (effects (font (size 1.27 1.27)) (justify right))
     )
-    (property "Footprint" "footprints:Liansheng FH-00357" (id 2) (at 123.19 60.96 0)
+    (property "Footprint" "footprints:Ckmtw_B-3000N34P-0110" (id 2) (at 123.19 60.96 0)
       (effects (font (size 1.27 1.27)) hide)
     )
@@
       (effects (font (size 1.27 1.27)) hide)
     )
-    (property "LCSC" "C2685114" (id 4) (at 123.19 60.96 90)
+    (property "LCSC" "C383613" (id 4) (at 123.19 60.96 90)
       (effects (font (size 1.27 1.27)) hide)
     )
@@
     )
     (path "/2690810c-9e74-4209-b5b4-4a1abf5844a3"
-      (reference "J2") (unit 1) (value "Conn_02x17_Odd_Even") (footprint "footprints:Liansheng FH-00357")
+      (reference "J2") (unit 1) (value "Conn_02x17_Odd_Even") (footprint "footprints:Ckmtw_B-3000N34P-0110")
     )
   )

Commit message: JLCPCB denied my part request; now they have to solder it by hand (THT)
Parts:
- J2: footprint footprints:Ckmtw_B-3000N34P-0110 -> footprints:JILN_321034SG0ABK00A01; LCSC C383613 -> C601943
Changed lines of the file:
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@@
       (effects (font (size 1.27 1.27)) (justify right))
     )
-    (property "Footprint" "footprints:Ckmtw_B-3000N34P-0110" (id 2) (at 123.19 60.96 0)
+    (property "Footprint" "footprints:JILN_321034SG0ABK00A01" (id 2) (at 123.19 60.96 0)
       (effects (font (size 1.27 1.27)) hide)
     )
@@
       (effects (font (size 1.27 1.27)) hide)
     )
-    (property "LCSC" "C383613" (id 4) (at 123.19 60.96 90)
+    (property "LCSC" "C601943" (id 4) (at 123.19 60.96 90)
       (effects (font (size 1.27 1.27)) hide)
     )
@@
     )
     (path "/2690810c-9e74-4209-b5b4-4a1abf5844a3"
-      (reference "J2") (unit 1) (value "Conn_02x17_Odd_Even") (footprint "footprints:Ckmtw_B-3000N34P-0110")
+      (reference "J2") (unit 1) (value "Conn_02x17_Odd_Even") (footprint "footprints:JILN_321034SG0ABK00A01")
     )
   )

Commit message: turn small connector into THT as well
Parts:
- J1: footprint footprints:XFCN MF254VS-11-06P-A -> footprints:Boom_Precision_Elec_C40877; LCSC C492238 -> C40877
Changed lines of the file:
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@@
       (effects (font (size 1.27 1.27)) (justify left))
     )
-    (property "Footprint" "footprints:XFCN MF254VS-11-06P-A" (id 2) (at 175.26 62.23 0)
+    (property "Footprint" "footprints:Boom_Precision_Elec_C40877" (id 2) (at 175.26 62.23 0)
       (effects (font (size 1.27 1.27)) hide)
     )
@@
       (effects (font (size 1.27 1.27)) hide)
     )
-    (property "LCSC" "C492238" (id 4) (at 175.26 62.23 0)
+    (property "LCSC" "C40877" (id 4) (at 175.26 62.23 0)
       (effects (font (size 1.27 1.27)) hide)
     )
@@
   (symbol_instances
     (path "/b571620c-4d41-45f5-a2f5-6e896d1e6a4a"
-      (reference "J1") (unit 1) (value "Conn_01x06") (footprint "footprints:XFCN MF254VS-11-06P-A")
+      (reference "J1") (unit 1) (value "Conn_01x06") (footprint "footprints:Boom_Precision_Elec_C40877")
     )
     (path "/2690810c-9e74-4209-b5b4-4a1abf5844a3"
